Commit message: Go Chase it

File: Go-Chase-it/my_robot/urdf/my_robot.xacro (robot description, xacro)
@@ -1,4 +1,5 @@
 <?xml version='1.0'?>
 <robot name="my_robot" xmlns:xacro="http://www.ros.org/wiki/xacro">
+<xacro:include filename="$(find my_robot)/urdf/my_robot.gazebo" />
   <link name="robot_footprint"></link>
   <joint name="robot_footprint_joint" type="fixed">
@@ -7,4 +8,5 @@
     <child link="chassis" />
   </joint>
+  <!-- #################### Chasis x = 0.6    y = 0.3   z = 0.1 ######################## -->
   <link name='chassis'>
     <pose>0 0 0.1 0 0 0</pose>
@@ -55,4 +57,63 @@
     </visual>
   </link>
+  <!-- #################### Camera & Lidar ######################## -->
+  <link name="camera">
+    <inertial>
+      <mass value="0.1"/>
+      <origin xyz="0 0 0" rpy="0 0 3.14" />
+      <inertia
+        ixx="0.1" ixy="0" ixz="0"
+        iyy="0.1" iyz="0"
+        izz="0.1"
+      />
+    </inertial>
+    <visual name="visual_camera">
+      <origin xyz="0 0 0" rpy=" 0 0 3.14"/>
+      <geometry>
+        <mesh filename="package://my_robot/meshes/camera.dae" scale="0.01 0.01 0.015"/>
+      </geometry>
+    </visual>
+    <collision>
+      <origin xyz="0 0 0" rpy=" 0 0 0"/>
+      <geometry>
+        <box size=".1 .1 .1"/>
+      </geometry>
+    </collision>
+  </link>
+  <link name="hokuyo">
+    <inertial>
+      <mass value="0.1"/>
+      <origin xyz="0 0 0.125" rpy="0 0 0" />
+      <inertia
+        ixx="0" ixy="0" ixz="0"
+        iyy="0" iyz="0" izz="0"
+      />
+    </inertial>
+    <visual>
+      <origin xyz="0 0 0" rpy=" 0 0 0"/>
+      <geometry>
+        <mesh filename = "package://my_robot/meshes/hokuyo.dae"/>
+      </geometry>
+    </visual>
+    <collision>
+      <origin xyz="0 0 0" rpy=" 0 0 0"/>
+      <geometry>
+        <box size=".1 .1 .1"/>
+      </geometry>
+    </collision>
+  </link>
+  <joint name="JOINT_camera" type="fixed">
+    <parent link="robot_footprint"/>
+    <child link="camera"/>
+    <origin xyz="0.33 0 0" rpy="0 0 0" />
+    <axis xyz="1 0 0" rpy="0 0 0"/>
+  </joint>
+  <joint name="JOINT_lidar" type="fixed">
+    <parent link="robot_footprint"/>
+    <child link="hokuyo"/>
+    <origin xyz="0.2 0 0.05" rpy="0 0 0" />
+    <axis xyz="1 0 0" rpy="0 0 0"/>
+  </joint>
+  <!-- #################### Wheels ######################## -->
   <link name="front_left_wheel">
     <pose>0 0 0 0 0 0</pose>
@@ -69,5 +130,5 @@
       <origin xyz="0 0 0" rpy=" 0 1.5707 1.5707"/>
       <geometry>
-        <cylinder radius="0.1" length="0.05"/>
+        <mesh filename="package://my_robot/meshes/wheel.dae" scale="0.03 0.03 0.03"/>
       </geometry>
     </visual>
@@ -83,4 +144,28 @@
     <inertial>
       <mass value="5.0"/>
+      <origin xyz="0.0 0 0" rpy=" 3.14 1.5707 1.5707"/>
+      <inertia
+          ixx="0.1" ixy="0" ixz="0"
+          iyy="0.1" iyz="0"
+          izz="0.1"
+      />
+    </inertial>
+    <visual>
+      <origin xyz="0 0 0" rpy=" 3.14 1.5707 1.5707"/>
+      <geometry>
+        <mesh filename="package://my_robot/meshes/wheel.dae" scale="0.03 0.03 0.03"/>
+      </geometry>
+    </visual>
+    <collision>
+      <origin xyz="0 0 0" rpy=" 0 1.5707 1.5707"/>
+      <geometry>
+        <cylinder radius="0.1" length="0.05"/>
+      </geometry>
+    </collision>
+  </link>
+  <link name="back_left_wheel">
+    <pose>0 0 0 0 0 0</pose>
+    <inertial>
+      <mass value="5.0"/>
       <origin xyz="0.0 0 0" rpy=" 0 1.5707 1.5707"/>
       <inertia
@@ -93,29 +178,5 @@
       <origin xyz="0 0 0" rpy=" 0 1.5707 1.5707"/>
       <geometry>
-        <cylinder radius="0.1" length="0.05"/>
-      </geometry>
-    </visual>
-    <collision>
-      <origin xyz="0 0 0" rpy=" 0 1.5707 1.5707"/>
-      <geometry>
-        <cylinder radius="0.1" length="0.05"/>
-      </geometry>
-    </collision>
-  </link>
-  <link name="back_left_wheel">
-    <pose>0 0 0 0 0 0</pose>
-    <inertial>
-      <mass value="5.0"/>
-      <origin xyz="0.0 0 0" rpy=" 0 1.5707 1.5707"/>
-      <inertia
-          ixx="0.1" ixy="0" ixz="0"
-          iyy="0.1" iyz="0"
-          izz="0.1"
-      />
-    </inertial>
-    <visual>
-      <origin xyz="0 0 0" rpy=" 0 1.5707 1.5707"/>
-      <geometry>
-        <cylinder radius="0.1" length="0.05"/>
+        <mesh filename="package://my_robot/meshes/wheel.dae" scale="0.03 0.03 0.03"/>
       </geometry>
     </visual>
@@ -131,15 +192,15 @@
     <inertial>
       <mass value="5.0"/>
-      <origin xyz="0.0 0 0" rpy=" 0 1.5707 1.5707"/>
-      <inertia
-          ixx="0.1" ixy="0" ixz="0"
-          iyy="0.1" iyz="0"
-          izz="0.1"
-      />
-    </inertial>
-    <visual>
-      <origin xyz="0 0 0" rpy=" 0 1.5707 1.5707"/>
-      <geometry>
-        <cylinder radius="0.1" length="0.05"/>
+      <origin xyz="0.0 0 0" rpy=" 3.14 1.5707 1.5707"/>
+      <inertia
+          ixx="0.1" ixy="0" ixz="0"
+          iyy="0.1" iyz="0"
+          izz="0.1"
+      />
+    </inertial>
+    <visual>
+      <origin xyz="0 0 0" rpy=" 3.14 1.5707 1.5707"/>
+      <geometry>
+        <mesh filename="package://my_robot/meshes/wheel.dae" scale="0.03 0.03 0.03"/>
       </geometry>
     </visual>
